Commit message: modify config

File: SC-LIO-SAM/launch/include/config/robot.urdf.xacro (robot description, xacro)
@@ -15,8 +15,20 @@
     <origin xyz="0 0 0" rpy="0 0 0" />
   </joint>
+  <link name="livox_frame"> </link>
+  <joint name="livox_frame_joint" type="fixed">
+    <parent link="chassis_link" />
+    <child link="livox_frame" />
+    <origin xyz="0 0 0" rpy="0 0 0" />
+  </joint>
   <link name="velodyne"> </link>
   <joint name="velodyne_joint" type="fixed">
     <parent link="chassis_link" />
     <child link="velodyne" />
+    <origin xyz="0 0 0" rpy="0 0 0" />
+  </joint>
+  <link name="rslidar"> </link>
+  <joint name="rslidar_joint" type="fixed">
+    <parent link="chassis_link" />
+    <child link="rslidar" />
     <origin xyz="0 0 0" rpy="0 0 0" />
   </joint>
